Commit message: change something

File: robotv1_description/urdf/gripper.xacro (robot description, xacro)
@@ -15,9 +15,9 @@
       </visual>
       <inertial>
-        <mass value=".001"/>
+        <mass value=".01"/>
         <inertia
-          ixx="0.001" ixy="0.0" ixz="0.0"
-          iyy="0.001" iyz="0.0"
-          izz="0.001"/>
+          ixx="0.0001" ixy="0.0" ixz="0.0"
+          iyy="0.0001" iyz="0.0"
+          izz="0.0001"/>
       </inertial>
     </link>
@@ -37,9 +37,9 @@
       </visual>
       <inertial>
-        <mass value="0.0001"/>
+        <mass value="0.01"/>
         <inertia
-          ixx="0.001" ixy="0.0" ixz="0.0"
-          iyy="0.001" iyz="0.0"
-          izz="0.001"/>
+          ixx="0.0001" ixy="0.0" ixz="0.0"
+          iyy="0.0001" iyz="0.0"
+          izz="0.0001"/>
       </inertial>
     </link>
@@ -56,9 +56,9 @@
       </visual>
       <inertial>
-        <mass value="0.0001"/>
+        <mass value="0.01"/>
         <inertia
-          ixx="0.001" ixy="0.0" ixz="0.0"
-          iyy="0.001" iyz="0.0"
-          izz="0.001"/>
+          ixx="0.0001" ixy="0.0" ixz="0.0"
+          iyy="0.0001" iyz="0.0"
+          izz="0.0001"/>
       </inertial>
     </link>
@@ -78,9 +78,9 @@
     </visual>
       <inertial>
-        <mass value="0.0001"/>
+        <mass value="0.01"/>
         <inertia
-          ixx="0.001" ixy="0.0" ixz="0.0"
-          iyy="0.001" iyz="0.0"
-          izz="0.001"/>
+          ixx="0.0001" ixy="0.0" ixz="0.0"
+          iyy="0.0001" iyz="0.0"
+          izz="0.0001"/>
       </inertial>
     </link>
@@ -97,9 +97,9 @@
       </visual>
       <inertial>
-        <mass value="0.0001"/>
+        <mass value="0.01"/>
         <inertia
-          ixx="0.001" ixy="0.0" ixz="0.0"
-          iyy="0.001" iyz="0.0"
-          izz="0.001"/>
+          ixx="0.0001" ixy="0.0" ixz="0.0"
+          iyy="0.0001" iyz="0.0"
+          izz="0.0001"/>
       </inertial>
     </link>

File: robotv1_description/urdf/leg.xacro (robot description, xacro)
@@ -23,5 +23,5 @@
   <xacro:property name="lenx_foot" value="0.1"/>
   <xacro:property name="leny_foot" value="0.04"/>
-  <xacro:property name="lenz_foot" value="0.002"/>
+  <xacro:property name="lenz_foot" value="0.02"/>
   <xacro:property name="base_pos" value="${lenz_hip_3+lenz_upp_leg+lenz_low_leg+lenz_ang_2/2+lenz_foot}"/>
   <xacro:include filename="$(find robotv1_description)/urdf/leg.gazebo" />

File: robotv1_description/urdf/robotv1.urdf (robot description, URDF)
Before this commit: robot robotv1, 25 links, 24 joints
Links:
- link leftarm_left_finger: mass 0.0001 -> 0.001
- link leftarm_left_tip: mass 0.0001 -> 0.001
- link leftarm_right_finger: mass 0.0001 -> 0.001
- link leftarm_right_tip: mass 0.0001 -> 0.001
- link leftleg_foot: mass 0.0216 -> 0.216; geometry collision box size=0.1 0.04 0.02; visual box size=0.1 0.04 0.02
- link pelvis: mass 2.0736 -> 0.7776; geometry collision box size=0.06 0.12 0.04; visual box size=0.06 0.12 0.04
- link rightleg_foot: mass 0.0216 -> 0.216; geometry collision box size=0.1 0.04 0.02; visual box size=0.1 0.04 0.02
Joints:
- joint dummy_to_pelvis: origin xyz=0 0 0.5 rpy=0 0 0 -> xyz=0 0 0.33 rpy=0 0 0
- joint leftarm_shoulder_1_joint: origin xyz=0 0 0.03 -> xyz=0 0 0.02
- joint leftleg_hip_1_joint: origin xyz=0 0.08 0 -> xyz=0 0.06 0
- joint rightleg_hip_1_joint: origin xyz=0 -0.08 0 -> xyz=0 -0.06 0

File: robotv1_description/urdf/torso.xacro (robot description, xacro)
@@ -1,7 +1,7 @@
 <?xml version="1.0"?>
 <robot name="torso" xmlns:xacro="http://www.ros.org/wiki/xacro">
-  <xacro:property name="lenx_pelvis" value="0.08"/>
-  <xacro:property name="leny_pelvis" value="0.16"/>
-  <xacro:property name="lenz_pelvis" value="0.06"/>
+  <xacro:property name="lenx_pelvis" value="0.06"/>
+  <xacro:property name="leny_pelvis" value="0.12"/>
+  <xacro:property name="lenz_pelvis" value="0.04"/>
 <xacro:include filename="$(find robotv1_description)/urdf/utilities.xacro"/>
   <link name="pelvis" >
@@ -22,6 +22,6 @@
   </link>
   <gazebo reference="pelvis" >
-    <mu1>0.2</mu1>
-    <mu2>0.2</mu2>
+    <mu1>0.4</mu1>
+    <mu2>0.4</mu2>
     <material>Gazebo/White</material>
   </gazebo>

File: robotv1_description/urdf/utilities.xacro (robot description, xacro)
@@ -7,7 +7,7 @@
       <mass value="${mass}" />
       <inertia
-      ixx="${100*mass*(lenz*lenz+leny*leny)/12}" ixy="0.0" ixz="0.0"
-      iyy="${100*mass*(lenz*lenz+leny*leny)/12}" iyz="0.0"
-      izz="${100*mass*(lenz*lenz+leny*leny)/12}" />
+      ixx="${mass*(lenz*lenz+leny*leny)/12.0}" ixy="0.0" ixz="0.0"
+      iyy="${mass*(lenz*lenz+lenx*lenx)/12.0}" iyz="0.0"
+      izz="${mass*(lenx*lenx+leny*leny)/12.0}" />
     </inertial>
   </xacro:macro>
