Commit message: modified

File: robotv1_description/urdf/leg.xacro (robot description, xacro)
@@ -24,4 +24,5 @@
   <xacro:property name="leny_foot" value="0.04"/>
   <xacro:property name="lenz_foot" value="0.002"/>
+  <xacro:property name="base_pos" value="${lenz_hip_3+lenz_upp_leg+lenz_low_leg+lenz_ang_2/2+lenz_foot}"/>
   <xacro:include filename="$(find robotv1_description)/urdf/leg.gazebo" />
   <xacro:include filename="$(find robotv1_description)/urdf/utilities.xacro"/>

File: robotv1_description/urdf/robotv1.urdf (robot description, URDF)
Before this commit: robot robotv1, 9 links, 8 joints
Links:
- removed link right_leg_ang_1
- removed link right_leg_ang_2
- removed link right_leg_foot
- removed link right_leg_hip_2
- removed link right_leg_hip_3
- removed link right_leg_low_leg
- removed link right_leg_upp_leg
- added link leftarm_gripper, mass .001; visual box size=0.06 0.03 0.04
- added link leftarm_left_finger, mass 0.0001; visual mesh filename=package://urdf_tutorial/meshes/l_finger.dae
- added link leftarm_left_tip, mass 0.0001; visual mesh filename=package://urdf_tutorial/meshes/l_finger_tip.dae
- added link leftarm_low_arm, mass 0.1512; collision box size=0.02 0.04 0.07; visual box size=0.02 0.04 0.07
- added link leftarm_right_finger, mass 0.0001; visual mesh filename=package://urdf_tutorial/meshes/l_finger.dae
- added link leftarm_right_tip, mass 0.0001; visual mesh filename=package://urdf_tutorial/meshes/l_finger_tip.dae
- added link leftarm_sho, mass 0.1944; collision box size=0.06 0.03 0.04; visual box size=0.06 0.03 0.04
- added link leftarm_upp_arm, mass 0.3888; collision box size=0.02 0.06 0.12; visual box size=0.02 0.06 0.12
- added link leftarm_wri_1, mass 0.1944; collision box size=0.04 0.06 0.03; visual box size=0.04 0.06 0.03
- added link leftleg_ang_1, mass 0.1944; collision box size=0.04 0.03 0.06; visual box size=0.04 0.03 0.06
- added link leftleg_ang_2, mass 0.1944; collision box size=0.03 0.04 0.06; visual box size=0.03 0.04 0.06
- added link leftleg_foot, mass 0.0216; collision box size=0.1 0.04 0.002; visual box size=0.1 0.04 0.002
- added link leftleg_hip_2, mass 0.1944; collision box size=0.04 0.03 0.06; visual box size=0.04 0.03 0.06
- added link leftleg_hip_3, mass 0.5103; collision box size=0.07 0.03 0.09; visual box size=0.07 0.03 0.09
- added link leftleg_low_leg, mass 0.1404; collision box size=0.02 0.02 0.13; visual box size=0.02 0.02 0.13
- added link leftleg_upp_leg, mass 0.1944; collision box size=0.03 0.04 0.06; visual box size=0.03 0.04 0.06
- added link rightleg_ang_1, mass 0.1944; collision box size=0.04 0.03 0.06; visual box size=0.04 0.03 0.06
- added link rightleg_ang_2, mass 0.1944; collision box size=0.03 0.04 0.06; visual box size=0.03 0.04 0.06
- added link rightleg_foot, mass 0.0216; collision box size=0.1 0.04 0.002; visual box size=0.1 0.04 0.002
- added link rightleg_hip_2, mass 0.1944; collision box size=0.04 0.03 0.06; visual box size=0.04 0.03 0.06
- added link rightleg_hip_3, mass 0.5103; collision box size=0.07 0.03 0.09; visual box size=0.07 0.03 0.09
- added link rightleg_low_leg, mass 0.1404; collision box size=0.02 0.02 0.13; visual box size=0.02 0.02 0.13
- added link rightleg_upp_leg, mass 0.1944; collision box size=0.03 0.04 0.06; visual box size=0.03 0.04 0.06
Joints:
- removed joint right_leg_ang_1_joint
- removed joint right_leg_ang_2_joint
- removed joint right_leg_foot_joint
- removed joint right_leg_hip_1_joint
- removed joint right_leg_hip_2_joint
- removed joint right_leg_hip_3_joint
- removed joint right_leg_knee_joint
- added joint leftarm_elbow_joint: type revolute, parent leftarm_upp_arm, child leftarm_low_arm, origin xyz=0 0 0.12, axis 0 1 0, limit lower=0 upper=3.14159265359 effort=0.2 velocity=1.0
- added joint leftarm_left_finger_joint: type revolute, parent leftarm_gripper, child leftarm_left_finger, origin xyz=0.0 0.01 0 rpy=0 -1.57079632679 0, axis 0 0 1, limit lower=0 upper=0.785398163397 effort=0.0001 velocity=0.0001
- added joint leftarm_left_tip_joint: type fixed, parent leftarm_left_finger, child leftarm_left_tip
- added joint leftarm_right_finger_joint: type revolute, parent leftarm_gripper, child leftarm_right_finger, origin xyz=0.0 -0.01 0 rpy=0 -1.57079632679 0, axis 0 0 1, limit lower=-0.785398163397 upper=0 effort=0.0001 velocity=0.0001
- added joint leftarm_right_tip_joint: type fixed, parent leftarm_right_finger, child leftarm_right_tip
- added joint leftarm_shoulder_1_joint: type revolute, parent pelvis, child leftarm_sho, origin xyz=0 0 0.03, axis 0 0 1, limit lower=-1.57079632679 upper=1.57079632679 effort=0.2 velocity=1.0
- added joint leftarm_shoulder_2_joint: type revolute, parent leftarm_sho, child leftarm_upp_arm, origin xyz=0 0 0.02, axis 0 1 0, limit lower=-1.57079632679 upper=1.57079632679 effort=0.2 velocity=1.0
- added joint leftarm_wrist_1_joint: type revolute, parent leftarm_low_arm, child leftarm_wri_1, origin xyz=0 0 0.07, axis 0 1 0, limit lower=-1.57079632679 upper=1.57079632679 effort=0.2 velocity=1.0
- added joint leftarm_wrist_2_joint: type revolute, parent leftarm_wri_1, child leftarm_gripper, origin xyz=0 0 0.03, axis 0 0 1, limit lower=-1.57079632679 upper=1.57079632679 effort=0.2 velocity=1.0
- added joint leftleg_ang_1_joint: type revolute, parent leftleg_low_leg, child leftleg_ang_1, origin xyz=0 0 -0.1 rpy=0 0 0, axis 1 0 0, limit lower=-0.785398163397 upper=0.785398163397 effort=2 velocity=1.0
- added joint leftleg_ang_2_joint: type revolute, parent leftleg_ang_1, child leftleg_ang_2, origin xyz=-0.02 0 0, axis 0 1 0, limit lower=-0.785398163397 upper=0.785398163397 effort=2 velocity=1.0
- added joint leftleg_foot_joint: type fixed, parent leftleg_ang_2, child leftleg_foot, origin xyz=0 0 -0.06
- added joint leftleg_hip_1_joint: type revolute, parent pelvis, child leftleg_hip_2, origin xyz=0 0.08 0, axis 0 1 0, limit lower=-1.57079632679 upper=1.57079632679 effort=2 velocity=1.0
- added joint leftleg_hip_2_joint: type revolute, parent leftleg_hip_2, child leftleg_hip_3, origin xyz=0 0.03 0, axis 1 0 0, limit lower=-1.57079632679 upper=1.57079632679 effort=2 velocity=1.0
- added joint leftleg_hip_3_joint: type revolute, parent leftleg_hip_3, child leftleg_upp_leg, origin xyz=0 0 -0.09, axis 0 0 1, limit lower=-1.57079632679 upper=1.57079632679 effort=2 velocity=1.0
- added joint leftleg_knee_joint: type revolute, parent leftleg_upp_leg, child leftleg_low_leg, origin xyz=0 0 -0.06, axis 0 1 0, limit lower=0 upper=2.74889357189 effort=2 velocity=1.0
- added joint rightleg_ang_1_joint: type revolute, parent rightleg_low_leg, child rightleg_ang_1, origin xyz=0 0 -0.1 rpy=0 0 0, axis 1 0 0, limit lower=-0.785398163397 upper=0.785398163397 effort=2 velocity=1.0
- added joint rightleg_ang_2_joint: type revolute, parent rightleg_ang_1, child rightleg_ang_2, origin xyz=-0.02 0 0, axis 0 1 0, limit lower=-0.785398163397 upper=0.785398163397 effort=2 velocity=1.0
- added joint rightleg_foot_joint: type fixed, parent rightleg_ang_2, child rightleg_foot, origin xyz=0 0 -0.06
- added joint rightleg_hip_1_joint: type revolute, parent pelvis, child rightleg_hip_2, origin xyz=0 -0.08 0, axis 0 1 0, limit lower=-1.57079632679 upper=1.57079632679 effort=2 velocity=1.0
- added joint rightleg_hip_2_joint: type revolute, parent rightleg_hip_2, child rightleg_hip_3, origin xyz=0 -0.03 0, axis 1 0 0, limit lower=-1.57079632679 upper=1.57079632679 effort=2 velocity=1.0
- added joint rightleg_hip_3_joint: type revolute, parent rightleg_hip_3, child rightleg_upp_leg, origin xyz=0 0 -0.09, axis 0 0 1, limit lower=-1.57079632679 upper=1.57079632679 effort=2 velocity=1.0
- added joint rightleg_knee_joint: type revolute, parent rightleg_upp_leg, child rightleg_low_leg, origin xyz=0 0 -0.06, axis 0 1 0, limit lower=0 upper=2.74889357189 effort=2 velocity=1.0

File: robotv1_description/urdf/robotv1.xacro (robot description, xacro)
@@ -9,5 +9,5 @@
 <link name="dummy"/>
 <joint name="dummy_to_pelvis" type="fixed">
-  <origin xyz="0 0 0.5" rpy="0 0 0"/>
+  <origin xyz="0 0 ${base_pos}" rpy="0 0 0"/>
   <parent link="dummy" />
   <child link="pelvis" />

Commit message: test

File: robotv1_description/urdf/leg.xacro (robot description, xacro)
@@ -33,5 +33,5 @@
       <origin xyz="0 ${leny_pelvis*reflect/2} 0"/>
       <axis xyz="0 1 0"/>
-      <dynamics damping="0.7"/>
+      <dynamics damping="0.9"/>
       <limit effort="2" velocity="1.0" lower="${-pi/2}" upper="${pi/2}" />
     </joint>
@@ -57,5 +57,5 @@
       <origin xyz= "0 ${leny_hip_2*reflect} 0"/>
       <axis xyz="1 0 0"/>
-      <dynamics damping="0.7"/>
+      <dynamics damping="0.9"/>
       <limit effort="2" velocity="1.0" lower="${-pi/2}" upper="${pi/2}" />
     </joint>
@@ -81,5 +81,5 @@
       <origin xyz="0 0 ${-lenz_hip_3}"/>
       <axis xyz="0 0 1"/>
-      <dynamics damping="0.7"/>
+      <dynamics damping="0.9"/>
       <limit effort="2" velocity="1.0" lower="${-pi/2}" upper="${pi/2}" />
     </joint>
@@ -105,5 +105,5 @@
       <origin xyz="0 0 ${-lenz_upp_leg}"/>
       <axis xyz="0 1 0"/>
-      <dynamics damping="0.7"/>
+      <dynamics damping="0.9"/>
       <limit effort="2" velocity="1.0" lower="0" upper="${7*pi/8}" />
     </joint>
@@ -129,5 +129,5 @@
       <origin xyz="0 0 ${-lenz_low_leg+lenz_ang_1/2}" rpy="0 0 0"/>
       <axis xyz="1 0 0"/>
-      <dynamics damping="0.7"/>
+      <dynamics damping="0.9"/>
       <limit effort="2" velocity="1.0" lower="${-pi/4}" upper="${pi/4}" />
     </joint>
@@ -153,5 +153,5 @@
        <origin xyz="${-lenx_ang_1/2} 0 0"/>
        <axis xyz="0 1 0"/>
-       <dynamics damping="0.7"/>
+       <dynamics damping="0.9"/>
        <limit effort="2" velocity="1.0" lower="${-pi/4}" upper="${pi/4}" />
      </joint>
